File: circuit_board/_autosave-circuit_board.kicad_pcb (KiCad board)
At the start: 2 copper layers, 18 x 22.5 mm, 51 parts, among them J1 USB_C_Receptacle_USB2.0_16P, K1 SW_Omron_B3FS, K2 SW_Omron_B3FS, U1 ESP32-C3, Y1 NX3225SA-40M-EXS00A-CS03880

Commit message: backups save lives
Parts:
- added C3: Antenna, RF_Antenna:Johanson_2450AT43F0100, F.Cu at (179.4, 86.0)
- added D2: LED, LED_SMD:LED_0603_1608Metric, F.Cu at (194.2, 82.5)
- CD2: footprint SM0603UYC:LED_SM0603UYC -> LED_SMD:LED_0603_1608Metric
- moved CD2 16.4 mm to (194.8, 84.5), turned to -90 degrees
