File: circuit_board/_autosave-circuit_board.kicad_sch (KiCad schematic)
At the start: 46 parts, among them J1 USB_C_Receptacle_USB2.0_16P, J2 Conn_01x08_Pin, K1 SW_Omron_B3FS, K2 SW_Omron_B3FS, U1 ESP32-C3, Y1 NX3225SA-40M-EXS00A-CS03880

Commit message: backups save lives
Parts:
- removed CD1: LED, SM0603UYC:LED_SM0603UYC, symbol Device:LED
- removed J2: Conn_01x08_Pin, MountingHole:MountingHole_3.2mm_M3_DIN965_Pad, symbol Connector:Conn_01x08_Pin
- added D2: LED, LED_SMD:LED_0603_1608Metric, symbol Device:LED
- added H10: 6, Connector_Pin:Pin_D1.1mm_L8.5mm_W2.5mm_FlatFork, symbol Mechanical:MountingHole_Pad
- added H11: 4, Connector_Pin:Pin_D1.1mm_L8.5mm_W2.5mm_FlatFork, symbol Mechanical:MountingHole_Pad
- added H12: 2, Connector_Pin:Pin_D1.1mm_L8.5mm_W2.5mm_FlatFork, symbol Mechanical:MountingHole_Pad
- added H13: 7, Connector_Pin:Pin_D1.1mm_L8.5mm_W2.5mm_FlatFork, symbol Mechanical:MountingHole_Pad
- added H14: 5, Connector_Pin:Pin_D1.1mm_L8.5mm_W2.5mm_FlatFork, symbol Mechanical:MountingHole_Pad
- added H15: 3, Connector_Pin:Pin_D1.1mm_L8.5mm_W2.5mm_FlatFork, symbol Mechanical:MountingHole_Pad
- added H16: 1, Connector_Pin:Pin_D1.1mm_L8.5mm_W2.5mm_FlatFork, symbol Mechanical:MountingHole_Pad
- added H9: 8, Connector_Pin:Pin_D1.1mm_L8.5mm_W2.5mm_FlatFork, symbol Mechanical:MountingHole_Pad
- C3: footprint (none) -> Inductor_SMD:L_Wuerth_HCI-5040
- CD2: footprint SM0603UYC:LED_SM0603UYC -> LED_SMD:LED_0603_1608Metric
- H1, H2, H3, H4, H5, H6, H7, H8: footprint (none) -> Connector_Pin:Pin_D1.1mm_L8.5mm_W2.5mm_FlatFork
Connections:
- net GND: now also D2.1 (K)
- net GPIO10: now also H10.1
- net GPIO20: now also H13.1
- net GPIO21: now also H9.1
- net GPIO5/ADC2/SCL: now also H16.1
- net GPIO6: now also H12.1
- net GPIO7: now also H15.1
- net GPIO8/PWM: now also H11.1
- net GPIO9/BOOT: now also H14.1
- net at UR7.2: now also D2.2 (A)
