File: circuit_board/circuit_board.kicad_sch (KiCad schematic)
At the start: 39 parts, among them J1 USB_C_Receptacle_USB2.0_16P, J2 Conn_01x08_Pin, J3 Conn_01x08_Pin, K1 SW_Omron_B3FS, K2 SW_Omron_B3FS, U1 ESP32-C3, Y1 NX3225SA-40M-EXS00A-CS03880

Commit message: backups save lives
Parts:
- removed J2, J3: Conn_01x08_Pin, symbol Connector:Conn_01x08_Pin
- added H1, H16: 1, Connector_Pin:Pin_D1.1mm_L8.5mm_W2.5mm_FlatFork, symbol Mechanical:MountingHole_Pad
- added H10, H6: 6, Connector_Pin:Pin_D1.1mm_L8.5mm_W2.5mm_FlatFork, symbol Mechanical:MountingHole_Pad
- added H11, H4: 4, Connector_Pin:Pin_D1.1mm_L8.5mm_W2.5mm_FlatFork, symbol Mechanical:MountingHole_Pad
- added H12, H2: 2, Connector_Pin:Pin_D1.1mm_L8.5mm_W2.5mm_FlatFork, symbol Mechanical:MountingHole_Pad
- added H13, H7: 7, Connector_Pin:Pin_D1.1mm_L8.5mm_W2.5mm_FlatFork, symbol Mechanical:MountingHole_Pad
- added H14, H5: 5, Connector_Pin:Pin_D1.1mm_L8.5mm_W2.5mm_FlatFork, symbol Mechanical:MountingHole_Pad
- added H15, H3: 3, Connector_Pin:Pin_D1.1mm_L8.5mm_W2.5mm_FlatFork, symbol Mechanical:MountingHole_Pad
- added H8, H9: 8, Connector_Pin:Pin_D1.1mm_L8.5mm_W2.5mm_FlatFork, symbol Mechanical:MountingHole_Pad
- C1, C2, UC1, UC10, UC11, UC12, UC13, UC2, UC5, UC6, UC7, UC8, UC9: footprint Capacitor_SMD:C_0201_0603Metric -> GRM033R61E431KA01D:CAPC0603X33N
- CD1, CD2: footprint LED_SMD:LED_0201_0603Metric -> SM0603UYC:LED_SM0603UYC
- K1, K2: footprint Button_Switch_SMD:SW_Push_SPST_NO_Alps_SKRK -> SKRKAEE010:SKRK
- PC1, PC2, UC4: footprint Capacitor_SMD:C_0402_1005Metric -> C0402C152J5GACTU:CAPC1005X55N
- PU1: footprint Package_TO_SOT_SMD:SOT-23-5 -> LP3985IM5-3.3:SOT95P280X145-5N
- U1: footprint Package_DFN_QFN:QFN-32-1EP_5x5mm_P0.5mm_EP3.7x3.7mm -> ESP32C3:QFN32_5X5MM
- UR1, UR10, UR15, UR2, UR3, UR4, UR5, UR7, UR8, UR9: footprint Resistor_SMD:R_0201_0603Metric -> RC0201FR-0768KL:RESC0603X26N
- UR6: value R -> 10; footprint Resistor_SMD:R_0201_0603Metric -> RC0201FR-0768KL:RESC0603X26N
Connections:
- net +3.3V: now also H6.1
- net GND: now also H7.1
- net GPIO0/U1TXD: now also H1.1
- net GPIO10: now also H10.1
- net GPIO1/U1RXD: now also H2.1
- net GPIO2: now also H3.1
- net GPIO20: now also H13.1
- net GPIO21: now also H9.1
- net GPIO3: now also H4.1
- net GPIO4/ADC1/SDA: now also H5.1
- net GPIO5/ADC2/SCL: now also H16.1
- net GPIO6: now also H12.1
- net GPIO7: now also H15.1
- net GPIO8/PWM: now also H11.1
- net GPIO9/BOOT: now also H14.1
- net VBUS: now also H8.1
