File: circuit_board/circuit_board.kicad_pcb (KiCad board)
At the start: 2 copper layers, 18 x 22.5 mm, 51 parts, among them J1 USB_C_Receptacle_USB2.0_16P, K1 SW_Omron_B3FS, K2 SW_Omron_B3FS, U1 ESP32-C3, Y1 NX3225SA-40M-EXS00A-CS03880

Commit message: made a lot of changes
Parts:
- added C3: Antenna, Inductor_SMD:L_Wuerth_HCI-5040, F.Cu at (180.5, 85.7)
- added D2: LED, LED_SMD:LED_0603_1608Metric, F.Cu at (174.0, 70.3)
- CD2: footprint SM0603UYC:LED_SM0603UYC -> LED_SMD:LED_0603_1608Metric
- moved C1 47.6 mm to (173.5, 82.2), turned to 90 degrees
- moved PC1 46.6 mm to (174.0, 79.2)
- moved UR4 44.6 mm to (185.5, 67.8)
- moved PC2 44.3 mm to (179.7, 82.2), turned to 180 degrees
- moved C2 43.4 mm to (178.0, 81.7), turned to -90 degrees
- moved UC11 41.7 mm to (178.0, 75.0), turned to -90 degrees
- moved UR1 41.6 mm to (185.5, 68.5)
- moved UC12 40.7 mm to (185.5, 79.8)
- moved UC6 40.6 mm to (185.9, 78.9), turned to -90 degrees
- moved UC8 40.4 mm to (184.6, 82.2), turned to -90 degrees
- moved UC7 40.3 mm to (184.6, 80.2), turned to 90 degrees
- moved UR6 39.9 mm to (185.7, 69.7), turned to 180 degrees
- moved UR8 39.4 mm to (185.6, 74.4), turned to 90 degrees
- moved UC13 39.4 mm to (185.5, 80.5), turned to 180 degrees
- moved UC4 39.3 mm to (185.2, 82.0), turned to -90 degrees
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Routing:
- net GND: track 0.00 -> 71.2 mm, vias 0 -> 12
- net +3.3V: track 0.00 -> 53.1 mm, vias 0 -> 6
- net CHIP EN: track 0.00 -> 20.1 mm, vias 0 -> 3
- net GPIO7: track 0.00 -> 19.0 mm, vias 0 -> 1
- net GPIO6: track 0.00 -> 16.4 mm, vias 0 -> 3
- net GPIO8/PWM: track 0.00 -> 15.9 mm, vias 0 -> 1
- net Net-(J1-D--PadA7): track 0.00 -> 15.7 mm, vias 0 -> 4
- net VBUS: track 0.00 -> 15.0 mm
- net Net-(J1-D+-PadA6): track 0.00 -> 14.8 mm, vias 0 -> 5
- net VSYS: track 0.00 -> 14.1 mm, vias 0 -> 2
- net GPIO9/BOOT: track 0.00 -> 12.1 mm, vias 0 -> 1
- net GPIO10: track 0.00 -> 11.4 mm, vias 0 -> 1
- net GPIO2: track 0.00 -> 9.16 mm, vias 0 -> 1
- net CC2: track 0.00 -> 8.86 mm
- net GPIO0/U1TXD: track 0.00 -> 8.16 mm
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- added copper zone on B.Cu, net (none)
- added copper zone on F.Cu, net (none)
- removed copper zone on B.Cu, net GND
- removed copper zone on F.Cu, net GND
