File: circuit_board/circuit_v1/circuit_board.kicad_sch (KiCad schematic)
At the start: 46 parts, among them J1 USB_C_Receptacle_USB2.0_16P, J2 Conn_01x08_Pin, K1 SW_Omron_B3FS, K2 SW_Omron_B3FS, U1 ESP32-C3, Y1 NX3225SA-40M-EXS00A-CS03880

Commit message: backups save lives
Parts:
- removed C3: Antenna, symbol Device:Antenna
- removed H1: 1, symbol Mechanical:MountingHole_Pad
- removed H2: 2, symbol Mechanical:MountingHole_Pad
- removed H3: 3, symbol Mechanical:MountingHole_Pad
- removed H4: 4, symbol Mechanical:MountingHole_Pad
- removed H5: 5, symbol Mechanical:MountingHole_Pad
- removed H6: 6, symbol Mechanical:MountingHole_Pad
- removed H7: 7, symbol Mechanical:MountingHole_Pad
- removed H8: 8, symbol Mechanical:MountingHole_Pad
- added J3: Conn_01x08_Pin, symbol Connector:Conn_01x08_Pin
- added L1: L, Inductor_SMD:L_0201_0603Metric, symbol Device:L
- C1, C2, UC1, UC10, UC11, UC12, UC13, UC2, UC5, UC6, UC7, UC8, UC9: footprint GRM033R61E431KA01D:CAPC0603X33N -> Capacitor_SMD:C_0201_0603Metric
- J2: footprint MountingHole:MountingHole_3.2mm_M3_DIN965_Pad -> (none)
- K1, K2: footprint SKRKAEE010:SKRK -> Button_Switch_SMD:SW_Push_SPST_NO_Alps_SKRK
- PC1, PC2, UC4: footprint C0402C152J5GACTU:CAPC1005X55N -> Capacitor_SMD:C_0402_1005Metric
- PU1: footprint LP3985IM5-3.3:SOT95P280X145-5N -> Package_TO_SOT_SMD:SOT-23-5
- U1: footprint ESP32C3:QFN32_5X5MM -> Package_DFN_QFN:QFN-32-1EP_5x5mm_P0.5mm_EP3.7x3.7mm
- UR1, UR10, UR15, UR2, UR3, UR4, UR5, UR7, UR8, UR9: footprint RC0201FR-0768KL:RESC0603X26N -> Resistor_SMD:R_0201_0603Metric
- UR6: value 10 -> R; footprint RC0201FR-0768KL:RESC0603X26N -> Resistor_SMD:R_0201_0603Metric
Connections:
- net +3.3V: now also J3.6 (Pin_6)
- net GND: now also J3.7 (Pin_7)
- net GPIO0/U1TXD: now also J3.1 (Pin_1)
- net GPIO1/U1RXD: now also J3.2 (Pin_2)
- net GPIO2: now also J3.3 (Pin_3)
- net GPIO3: now also J3.4 (Pin_4)
- net GPIO4/ADC1/SDA: now also J3.5 (Pin_5)
- net VBUS: now also J3.8 (Pin_8)
- net at UC8.1, UR9.2: now also L1.1
- no-connect marks 8 -> 9
Other:
- company: Asfandyar Khan -> (none)
- title: ESP32-C3  -> (none)
- moved on the sheet: CD1, UC2, UR7
